File: Uguisu.kicad_sch (KiCad schematic)
At the start: 0 parts

Commit message: Restore KiCad schematic and PCB
Made-with: Cursor
Parts:
- added KEY1: SKQGABE010, easyeda2kicad:KEY-SMD_4P-L5.2-W5.2-P3.70-LS6.4, symbol easyeda2kicad:SKQGABE010
- added LED2: TC5050RGBF08-3CJH-AF53A, easyeda2kicad:LED-SMD_6P-L5.0-W5.0-TL_TC5050RGBF08, symbol easyeda2kicad:TC5050RGBF08-3CJH-AF53A
- added R1: 330, Resistor_SMD:R_0603_1608Metric, symbol Device:R
- added R2: 150, Resistor_SMD:R_0603_1608Metric, symbol Device:R
- added R3: 120, Resistor_SMD:R_0603_1608Metric, symbol Device:R
- added TP1: +BATT, TestPoint:TestPoint_Pad_3.0x3.0mm, symbol Connector:TestPoint
- added TP2: GND, TestPoint:TestPoint_Pad_3.0x3.0mm, symbol Connector:TestPoint
- added U1: XIAO-nRF52840-SMD, Seeed_Studio_XIAO_Series:XIAO-nRF52840-SMD, symbol Seeed_Studio_XIAO_Series:XIAO-nRF52840-SMD
Connections:
- new net: LED2.4 (-), R3.1
- new net: LED2.5 (-), R1.1
- new net: LED2.6 (-), R2.2
- new net +BATT: TP1.1, U1.32 (BAT)
- new net GND: KEY1.3, KEY1.4, TP2.1, U1.13 (GND), U1.27 (GND), U1.33 (GND)
- new net MCU_D0: KEY1.1, KEY1.2, U1.1 (P0.02_A0_D0)
- new net MCU_D1: R2.1, U1.2 (P0.03_A1_D1)
- new net MCU_D2: R1.2, U1.3 (P0.28_A2_D2)
- new net MCU_D3: R3.2, U1.4 (P0.29_A3_D3)
- no-connect marks 0 -> 14
