File: Guillemot/hardware/Guillemot.kicad_sch (KiCad schematic)
At the start: 34 parts, among them Q1 IPB042N10N3G, Q2 AO3422, Q3 SI2309CDS, Q4 2N7002, Q5 MMBT3904, Q6 MMBT3904, U1 XIAO-nRF52840-SMD, U2 SN74LVC2G02DCTR

Commit message: Update C2 to EMK325ABJ107MM-P, add no-hardware-edits rule, add codebase docs
- C2: EMK325ABJ107MM-P 100µF 16V X5R (was CL32A107MPVNNNE 10V)
- Cursor rule: do not modify files under hardware/
- Guillemot: KiCad schematic/PCB LCSC C90143, README, matched parts
- logs/18-CODEBASE_TECHNICAL_DOCUMENTATION.md

Made-with: Cursor
Parts:
- removed Q1: IPB042N10N3G, Package_TO_SOT_SMD:TO-263-2, symbol Transistor_FET:Q_NMOS_GDS
- added Q1: IPB042N10N3G, easyeda2kicad:TO-263-2_L10.0-W9.1-P5.08-LS15.2-TL, symbol easyeda2kicad:IPB042N10N3G
- C2: LCSC Part (none) -> C90143
Connections:
- net ESC-: now also Q1.4 (D)
- net GND: now also Q1.3 (S)
- net ISO_GATE: now also Q1.1 (G)
Changed lines of the file:
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@@
 	)
 	(label "ISO_GATE"
-		(at 182.88 83.82 180)
+		(at 189.23 68.58 180)
 		(effects
 			(font
@@
 	)
 	(label "ESC-"
-		(at 190.5 78.74 0)
+		(at 196.85 63.5 0)
 		(effects
 			(font
@@
 			)
 		)
+		(property "LCSC Part" "C90143"
+			(at 180.34 49.53 90)
+			(effects
+				(font
+					(size 1.27 1.27)
+				)
+				(hide yes)
+			)
+		)
 		(pin "2"
 		)
@@
 	)
 	(symbol
-		(lib_id "Transistor_FET:Q_NMOS_GDS")
-		(at 187.96 83.82 0)
-		(unit 1)
-		(exclude_from_sim no)
-		(in_bom yes)
-		(on_board yes)
-		(dnp no)
-		(property "Reference" "Q1"
-			(at 194.31 82.5499 0)
-			(effects
-				(font
-					(size 1.27 1.27)
-				)
-				(justify left)
-			)
-		)
-		(property "Value" "IPB042N10N3G"
-			(at 194.31 85.0899 0)
-			(effects
-				(font
-					(size 1.27 1.27)
-				)
-				(justify left)
-			)
-		)
-		(property "Footprint" "Package_TO_SOT_SMD:TO-263-2"
-			(at 193.04 81.28 0)
-			(effects
-				(font
-					(size 1.27 1.27)
-				)
-				(hide yes)
-			)
-		)
-		(property "Datasheet" "~"
-			(at 187.96 83.82 0)
-			(effects
-				(font
-					(size 1.27 1.27)
-				)
-				(hide yes)
-			)
-		)
-		(property "Description" "N-MOSFET transistor, gate/drain/source"
-			(at 187.96 83.82 0)
-			(effects
-				(font
-					(size 1.27 1.27)
-				)
-				(hide yes)
-			)
-		)
-		(property "LCSC Part" "C69300"
-			(at 187.96 83.82 0)
-			(effects
-				(font
-					(size 1.27 1.27)
-				)
-				(hide yes)
-			)
-		)
-		(pin "3"
-		)
-		(pin "2"
-		)
-		(pin "1"
-		)
-		(instances
-			(project ""
-				(path "/024e03f0-ce48-4a1e-8a44-0ff4b1918b95"
-					(reference "Q1")
-					(unit 1)
-				)
-			)
-		)
-	)
-	(symbol
 		(lib_id "Diode:1N4148")
 		(at 254 71.12 180)
@@
 	(symbol
 		(lib_id "power:GND")
-		(at 190.5 88.9 0)
+		(at 196.85 73.66 0)
 		(unit 1)
 		(exclude_from_sim no)
@@
 		(fields_autoplaced yes)
 		(property "Reference" "#PWR022"
-			(at 190.5 95.25 0)
+			(at 196.85 80.01 0)
 			(effects
 				(font
@@
 		)
 		(property "Value" "GND"
-			(at 190.5 93.98 0)
+			(at 196.85 78.74 0)
 			(effects
 				(font
@@
 		)
 		(property "Footprint" ""
-			(at 190.5 88.9 0)
+			(at 196.85 73.66 0)
 			(effects
 				(font
@@
 		)
 		(property "Datasheet" ""
-			(at 190.5 88.9 0)
+			(at 196.85 73.66 0)
 			(effects
 				(font
@@
 		)
 		(property "Description" "Power symbol creates a global label with name \"GND\" , ground"
-			(at 190.5 88.9 0)
+			(at 196.85 73.66 0)
 			(effects
 				(font
@@
 					(unit 1)
 				)
+			)
+		)
+	)
+	(symbol
+		(lib_id "easyeda2kicad:IPB042N10N3G")
+		(at 194.31 68.58 0)
+		(unit 1)
+		(exclude_from_sim no)
+		(in_bom yes)
+		(on_board yes)
+		(dnp no)
+		(fields_autoplaced yes)
+		(property "Reference" "Q1"
+			(at 201.93 67.3099 0)
+			(effects
+				(font
+					(size 1.27 1.27)
+				)
+				(justify left)
+			)
+		)
+		(property "Value" "IPB042N10N3G"
+			(at 201.93 69.8499 0)
+			(effects
+				(font
+					(size 1.27 1.27)
+				)
+				(justify left)
+			)
+		)
+		(property "Footprint" "easyeda2kicad:TO-263-2_L10.0-W9.1-P5.08-LS15.2-TL"
+			(at 194.31 81.28 0)
+			(effects
+				(font
+					(size 1.27 1.27)
+				)
+				(hide yes)
+			)
+		)
+		(property "Datasheet" "https://lcsc.com/product-detail/MOSFET_Infineon_IPB042N10N3G_IPB042N10N3G_C69300.html"
+			(at 194.31 83.82 0)
+			(effects
+				(font
+					(size 1.27 1.27)
+				)
+				(hide yes)
+			)
+		)
+		(property "Description" ""
+			(at 194.31 68.58 0)
+			(effects
+				(font
+					(size 1.27 1.27)
+				)
+				(hide yes)
+			)
+		)
+		(property "LCSC Part" "C69300"
+			(at 194.31 86.36 0)
+			(effects
+				(font
+					(size 1.27 1.27)
+				)
+				(hide yes)
+			)
+		)
+		(pin "3"
+		)
+		(pin "1"
+		)
+		(pin "4"
+		)
+		(instances
+			(project ""
+				(path "/024e03f0-ce48-4a1e-8a44-0ff4b1918b95"
+					(reference "Q1")
+					(unit 1)
+				)
